File: water_control/kicad/pond control 2.0.sch (KiCad schematic (older format))
At the start: 12 parts, among them J1 Conn_01x03_Male, J2 Conn_01x02_Male, J3 Conn_01x08_Male, Q1 TIP120, Q2 TIP120

Commit message: Added schematics
Parts:
- removed R4: 560, symbol Device:R
- added J?: Conn_01x04_Male, symbol Connector:Conn_01x04_Male
Connections:
- net +12V: now also J1.1 (Pin_1); no longer A1.30 (VIN), J1.2 (Pin_2)
- net +5V: now also J2.1 (Pin_1), J?.1 (Pin_1)
- net GND: now also J?.3 (Pin_3)
- net at A1.19 (A0): now also J?.2 (Pin_2), J?.4 (Pin_4); no longer J2.1 (Pin_1)
Other:
- note added: "GX12 - 2 wire\nTo RPI 4 (2.5-3A) adapter"
- note added: "GX12 - 3 wire (2 needed)\nFrom standard 12V transformer\n"
- note added: "GX12 - 4 wire\nKUS/etape level sensor"
- note added: "GX12 - 8 wire\nSolenoids and flow sensor"
- moved on the sheet: J1, J2
Changed lines of the file:
@@
 L Connector:Conn_01x02_Male J2
 U 1 1 60BFF19D
-P 8600 3300
-F 0 "J2" H 8572 3274 50  0000 R CNN
-F 1 "Conn_01x02_Male" H 8572 3183 50  0000 R CNN
-F 2 "" H 8600 3300 50  0001 C CNN
-F 3 "~" H 8600 3300 50  0001 C CNN
-	1    8600 3300
-	-1   0    0    -1
+P 2650 2550
+F 0 "J2" H 2650 2850 50  0000 R CNN
+F 1 "Conn_01x02_Male" H 2800 2700 50  0000 R CNN
+F 2 "" H 2650 2550 50  0001 C CNN
+F 3 "~" H 2650 2550 50  0001 C CNN
+	1    2650 2550
+	1    0    0    -1
 $EndComp
 $Comp
@@
 U 1 1 60BFFC2B
 P 9300 5350
-F 0 "J3" H 9272 5324 50  0000 R CNN
-F 1 "Conn_01x08_Male" H 9272 5233 50  0000 R CNN
+F 0 "J3" H 9450 5900 50  0000 R CNN
+F 1 "Conn_01x08_Male" H 9500 5800 50  0000 R CNN
 F 2 "" H 9300 5350 50  0001 C CNN
 F 3 "~" H 9300 5350 50  0001 C CNN
@@
 L Connector:Conn_01x03_Male J1
 U 1 1 60C0124F
-P 1950 2100
-F 0 "J1" H 2058 2381 50  0000 C CNN
-F 1 "Conn_01x03_Male" H 2058 2290 50  0000 C CNN
-F 2 "" H 1950 2100 50  0001 C CNN
-F 3 "~" H 1950 2100 50  0001 C CNN
-	1    1950 2100
-	1    0    0    -1
-$EndComp
-$Comp
-L power:+12V #PWR03
-U 1 1 60C0757E
-P 2700 2100
-F 0 "#PWR03" H 2700 1950 50  0001 C CNN
-F 1 "+12V" H 2715 2273 50  0000 C CNN
-F 2 "" H 2700 2100 50  0001 C CNN
-F 3 "" H 2700 2100 50  0001 C CNN
-	1    2700 2100
+P 2650 1550
+F 0 "J1" H 2758 1831 50  0000 C CNN
+F 1 "Conn_01x03_Male" H 2758 1740 50  0000 C CNN
+F 2 "" H 2650 1550 50  0001 C CNN
+F 3 "~" H 2650 1550 50  0001 C CNN
+	1    2650 1550
 	1    0    0    -1
 $EndComp
@@
 L power:GND #PWR02
 U 1 1 60C07D86
-P 2500 2300
-F 0 "#PWR02" H 2500 2050 50  0001 C CNN
-F 1 "GND" H 2505 2127 50  0000 C CNN
-F 2 "" H 2500 2300 50  0001 C CNN
-F 3 "" H 2500 2300 50  0001 C CNN
-	1    2500 2300
-	1    0    0    -1
-$EndComp
-Wire Wire Line
-	2150 2000 2500 2000
-Wire Wire Line
-	2500 2000 2500 1900
-Wire Wire Line
-	2150 2100 2700 2100
-Wire Wire Line
-	2150 2200 2500 2200
-Wire Wire Line
-	2500 2200 2500 2300
+P 3200 1750
+F 0 "#PWR02" H 3200 1500 50  0001 C CNN
+F 1 "GND" H 3205 1577 50  0000 C CNN
+F 2 "" H 3200 1750 50  0001 C CNN
+F 3 "" H 3200 1750 50  0001 C CNN
+	1    3200 1750
+	1    0    0    -1
+$EndComp
+Wire Wire Line
+	2850 1650 3200 1650
+Wire Wire Line
+	3200 1650 3200 1750
 $Comp
 L Device:R R1
@@
 	8900 5250 8900 5300
 $Comp
-L Device:R R4
-U 1 1 60C318B1
-P 7400 2950
-F 0 "R4" H 7330 2904 50  0000 R CNN
-F 1 "560" H 7330 2995 50  0000 R CNN
-F 2 "" V 7330 2950 50  0001 C CNN
-F 3 "~" H 7400 2950 50  0001 C CNN
-	1    7400 2950
-	-1   0    0    1
-$EndComp
-$Comp
 L power:+5V #PWR07
 U 1 1 60C32179
@@
 $EndComp
 Wire Wire Line
-	7400 2600 7400 2800
-Wire Wire Line
-	7400 3100 7400 3300
-Wire Wire Line
-	7400 3300 8400 3300
-Wire Wire Line
-	7400 3300 6500 3300
-Wire Wire Line
-	6500 3300 6500 3600
-Wire Wire Line
-	6500 3600 5900 3600
-Connection ~ 7400 3300
-Wire Wire Line
-	7400 3550 7400 3400
-Wire Wire Line
-	7400 3400 8400 3400
-Wire Wire Line
 	8300 5650 8550 5650
 Wire Wire Line
@@
 L power:+12V #PWR?
 U 1 1 60C3B09F
-P 5300 2450
-F 0 "#PWR?" H 5300 2300 50  0001 C CNN
-F 1 "+12V" H 5315 2623 50  0000 C CNN
-F 2 "" H 5300 2450 50  0001 C CNN
-F 3 "" H 5300 2450 50  0001 C CNN
-	1    5300 2450
+P 3200 1400
+F 0 "#PWR?" H 3200 1250 50  0001 C CNN
+F 1 "+12V" H 3215 1573 50  0000 C CNN
+F 2 "" H 3200 1400 50  0001 C CNN
+F 3 "" H 3200 1400 50  0001 C CNN
+	1    3200 1400
 	1    0    0    -1
 $EndComp
@@
 Wire Wire Line
 	5950 4600 5950 4650
+Wire Wire Line
+	2850 1450 3200 1450
+Wire Wire Line
+	3200 1450 3200 1400
+$Comp
+L power:+5V #PWR?
+U 1 1 62F3CBAE
+P 3200 2450
+F 0 "#PWR?" H 3200 2300 50  0001 C CNN
+F 1 "+5V" H 3215 2623 50  0000 C CNN
+F 2 "" H 3200 2450 50  0001 C CNN
+F 3 "" H 3200 2450 50  0001 C CNN
+	1    3200 2450
+	1    0    0    -1
+$EndComp
+$Comp
+L power:GND #PWR?
+U 1 1 62F3DE25
+P 3200 2800
+F 0 "#PWR?" H 3200 2550 50  0001 C CNN
+F 1 "GND" H 3205 2627 50  0000 C CNN
+F 2 "" H 3200 2800 50  0001 C CNN
+F 3 "" H 3200 2800 50  0001 C CNN
+	1    3200 2800
+	1    0    0    -1
+$EndComp
+Wire Wire Line
+	2850 2550 3200 2550
+Wire Wire Line
+	3200 2550 3200 2450
+Wire Wire Line
+	3200 2800 3200 2650
+Wire Wire Line
+	3200 2650 2850 2650
+$Comp
+L Connector:Conn_01x04_Male J?
+U 1 1 62F408FD
+P 9200 3050
+F 0 "J?" H 9550 3400 50  0000 R CNN
+F 1 "Conn_01x04_Male" H 9550 3300 50  0000 R CNN
+F 2 "" H 9200 3050 50  0001 C CNN
+F 3 "~" H 9200 3050 50  0001 C CNN
+	1    9200 3050
+	-1   0    0    -1
+$EndComp
+Wire Wire Line
+	5900 3600 6750 3600
+Wire Wire Line
+	6750 3600 6750 3250
+Wire Wire Line
+	6750 3050 9000 3050
+Wire Wire Line
+	9000 3150 7400 3150
+Wire Wire Line
+	7400 3150 7400 3550
+Wire Wire Line
+	9000 3250 6750 3250
+Connection ~ 6750 3250
+Wire Wire Line
+	6750 3250 6750 3050
+Wire Wire Line
+	9000 2950 7400 2950
+Wire Wire Line
+	7400 2950 7400 2600
+Text Notes 9400 3100 0    50   ~ 0
+GX12 - 4 wire\nKUS/etape level sensor
+Text Notes 9550 5400 0    50   ~ 0
+GX12 - 8 wire\nSolenoids and flow sensor
+Text Notes 1050 1550 0    50   ~ 0
+GX12 - 3 wire (2 needed)\nFrom standard 12V transformer\n
+Text Notes 1050 2700 0    50   ~ 0
+GX12 - 2 wire\nTo RPI 4 (2.5-3A) adapter
 $EndSCHEMATC
